Commit message: Inertia issue fixed

File: robot_arm_description/urdf/robot_arm.xacro (robot description, xacro)
@@ -4,4 +4,5 @@
 <xacro:include filename="$(find robot_arm_description)/urdf/robot_arm.trans" />
 <xacro:include filename="$(find robot_arm_description)/urdf/robot_arm.gazebo" />
+<link name="dummy"></link>
 <link name="base_link">
   <inertial>
@@ -124,4 +125,8 @@
   </collision>
 </link>
+<joint name="dummy_joint" type="fixed">
+  <parent link="dummy"/>
+  <child link="base_link"/>
+</joint>
 <joint name="base_rev" type="continuous">
   <origin rpy="0 0 0" xyz="0.0 0.0 0.057"/>
